Commit message: Fixed some labels and made positions consisent.

File: sim/spheres.urdf (robot description, URDF)
Before this commit: robot spheres, 5 links, 4 joints
Links:
- removed link obj_a
- removed link obj_b
- removed link obj_c
- removed link obj_d
- removed link obj_e
- added link s0, mass 0.0495; collision mesh filename=sphere_coll.obj scale=0.1 0.1 0.1; visual mesh filename=sphere.obj scale=0.1 0.1 0.1
- added link s1, mass 0.0495; collision mesh filename=sphere_coll.obj scale=0.1 0.1 0.1; visual mesh filename=sphere.obj scale=0.1 0.1 0.1
- added link s10, mass 0.0495; collision mesh filename=sphere_coll.obj scale=0.1 0.1 0.1; visual mesh filename=sphere.obj scale=0.1 0.1 0.1
- added link s11, mass 0.0495; collision mesh filename=sphere_coll.obj scale=0.1 0.1 0.1; visual mesh filename=sphere.obj scale=0.1 0.1 0.1
- added link s12, mass 0.0495; collision mesh filename=sphere_coll.obj scale=0.1 0.1 0.1; visual mesh filename=sphere.obj scale=0.1 0.1 0.1
- added link s13, mass 0.0495; collision mesh filename=sphere_coll.obj scale=0.1 0.1 0.1; visual mesh filename=sphere.obj scale=0.1 0.1 0.1
- added link s2, mass 0.0495; collision mesh filename=sphere_coll.obj scale=0.1 0.1 0.1; visual mesh filename=sphere.obj scale=0.1 0.1 0.1
- added link s3, mass 0.0495; collision mesh filename=sphere_coll.obj scale=0.1 0.1 0.1; visual mesh filename=sphere.obj scale=0.1 0.1 0.1
- added link s4, mass 0.0495; collision mesh filename=sphere_coll.obj scale=0.1 0.1 0.1; visual mesh filename=sphere.obj scale=0.1 0.1 0.1
- added link s5, mass 0.0495; collision mesh filename=sphere_coll.obj scale=0.1 0.1 0.1; visual mesh filename=sphere.obj scale=0.1 0.1 0.1
- added link s6, mass 0.0495; collision mesh filename=sphere_coll.obj scale=0.1 0.1 0.1; visual mesh filename=sphere.obj scale=0.1 0.1 0.1
- added link s7, mass 0.0495; collision mesh filename=sphere_coll.obj scale=0.1 0.1 0.1; visual mesh filename=sphere.obj scale=0.1 0.1 0.1
- added link s8, mass 0.0495; collision mesh filename=sphere_coll.obj scale=0.1 0.1 0.1; visual mesh filename=sphere.obj scale=0.1 0.1 0.1
- added link s9, mass 0.0495; collision mesh filename=sphere_coll.obj scale=0.1 0.1 0.1; visual mesh filename=sphere.obj scale=0.1 0.1 0.1
Joints:
- removed joint joint_sphere_a_b
- removed joint joint_sphere_b_c
- removed joint joint_sphere_c_d
- added joint joint_sphere_0_1: type revolute, parent s0, child s1, origin xyz=0.0 -0.4 0.0 rpy=0 0 0, axis 1 0 0, limit lower=-1.3963 upper=1.3963 effort=50000 velocity=10
- added joint joint_sphere_10_11: type revolute, parent s10, child s11, origin xyz=0.0 -0.4 0.0 rpy=0 0 0, axis 1 0 0, limit lower=-1.3963 upper=1.3963 effort=50000 velocity=10
- added joint joint_sphere_11_12: type revolute, parent s11, child s12, origin xyz=0.0 -0.4 0.0 rpy=0 0 0, axis 1 0 0, limit lower=-1.3963 upper=1.3963 effort=50000 velocity=10
- added joint joint_sphere_12_13: type revolute, parent s12, child s13, origin xyz=0.0 -0.4 0.0 rpy=0 0 0, axis 1 0 0, limit lower=-1.3963 upper=1.3963 effort=50000 velocity=10
- added joint joint_sphere_1_2: type revolute, parent s1, child s2, origin xyz=0.0 -0.4 0.0 rpy=0 0 0, axis 1 0 0, limit lower=-1.3963 upper=1.3963 effort=50000 velocity=10
- added joint joint_sphere_2_3: type revolute, parent s2, child s3, origin xyz=0.0 -0.4 0.0 rpy=0 0 0, axis 1 0 0, limit lower=-1.3963 upper=1.3963 effort=50000 velocity=10
- added joint joint_sphere_4_5: type revolute, parent s4, child s5, origin xyz=0.0 -0.4 0.0 rpy=0 0 0, axis 1 0 0, limit lower=-1.3963 upper=1.3963 effort=50000 velocity=10
- added joint joint_sphere_7_8: type revolute, parent s7, child s8, origin xyz=0.0 -0.4 0.0 rpy=0 0 0, axis 1 0 0, limit lower=-1.3963 upper=1.3963 effort=50000 velocity=10
- added joint joint_sphere_8_9: type revolute, parent s8, child s9, origin xyz=0.0 -0.4 0.0 rpy=0 0 0, axis 1 0 0, limit lower=-1.3963 upper=1.3963 effort=50000 velocity=10
- added joint joint_sphere_9_10: type revolute, parent s9, child s10, origin xyz=0.0 -0.4 0.0 rpy=0 0 0, axis 1 0 0, limit lower=-1.3963 upper=1.3963 effort=50000 velocity=10
- added joint joint_sphere_f_g: type revolute, parent s5, child s6, origin xyz=0.0 -0.4 0.0 rpy=0 0 0, axis 1 0 0, limit lower=-1.3963 upper=1.3963 effort=50000 velocity=10
- added joint joint_sphere_g_h: type revolute, parent s6, child s7, origin xyz=0.0 -0.4 0.0 rpy=0 0 0, axis 1 0 0, limit lower=-1.3963 upper=1.3963 effort=50000 velocity=10
- joint joint_sphere_d_e: axis (none) -> 1 0 0; child obj_e -> s4; parent obj_d -> s3

Commit message: [refactor] reduce reduce reduce.

File: sim/spheres.urdf (robot description, URDF)
Before this commit: robot spheres, 14 links, 13 joints
Joints:
- joint joint_sphere_0_1: limit lower=-1.3963 upper=1.3963 effort=50000 velocity=10 -> lower=-1.0467 upper=1.0467 effort=50000 velocity=10
- joint joint_sphere_10_11: limit lower=-1.3963 upper=1.3963 effort=50000 velocity=10 -> lower=-1.0467 upper=1.0467 effort=50000 velocity=10
- joint joint_sphere_11_12: limit lower=-1.3963 upper=1.3963 effort=50000 velocity=10 -> lower=-1.0467 upper=1.0467 effort=50000 velocity=10
- joint joint_sphere_12_13: limit lower=-1.3963 upper=1.3963 effort=50000 velocity=10 -> lower=-1.0467 upper=1.0467 effort=50000 velocity=10
- joint joint_sphere_1_2: limit lower=-1.3963 upper=1.3963 effort=50000 velocity=10 -> lower=-1.0467 upper=1.0467 effort=50000 velocity=10
- joint joint_sphere_2_3: limit lower=-1.3963 upper=1.3963 effort=50000 velocity=10 -> lower=-1.0467 upper=1.0467 effort=50000 velocity=10
- joint joint_sphere_4_5: limit lower=-1.3963 upper=1.3963 effort=50000 velocity=10 -> lower=-1.0467 upper=1.0467 effort=50000 velocity=10
- joint joint_sphere_7_8: limit lower=-1.3963 upper=1.3963 effort=50000 velocity=10 -> lower=-1.0467 upper=1.0467 effort=50000 velocity=10
- joint joint_sphere_8_9: limit lower=-1.3963 upper=1.3963 effort=50000 velocity=10 -> lower=-1.0467 upper=1.0467 effort=50000 velocity=10
- joint joint_sphere_9_10: limit lower=-1.3963 upper=1.3963 effort=50000 velocity=10 -> lower=-1.0467 upper=1.0467 effort=50000 velocity=10
- joint joint_sphere_d_e: limit lower=-1.3963 upper=1.3963 effort=50000 velocity=10 -> lower=-1.0467 upper=1.0467 effort=50000 velocity=10
- joint joint_sphere_f_g: limit lower=-1.3963 upper=1.3963 effort=50000 velocity=10 -> lower=-1.0467 upper=1.0467 effort=50000 velocity=10
- joint joint_sphere_g_h: limit lower=-1.3963 upper=1.3963 effort=50000 velocity=10 -> lower=-1.0467 upper=1.0467 effort=50000 velocity=10
